File: Layout/Powersupply.kicad_sch (KiCad schematic)
At the start: 0 parts

Commit message: Routine Commit, small changes in schematic
Parts:
- added C1, C2, C3, C4, C5, C6: C, symbol Device:C
- added J4: B2B-PH-K-S_LF__SN_, SHDR2W50P0X200_1X2_590X450X600P, symbol B2B-PH-K-S_LF__SN_:B2B-PH-K-S_LF__SN_
- added R1: R, symbol Device:R
- added U1: TP4056-42-ESOP8, Package_SO:SOIC-8-1EP_3.9x4.9mm_P1.27mm_EP2.41x3.3mm_ThermalVias, symbol Battery_Management:TP4056-42-ESOP8
- added U3, U4: XC6210B332MR, Package_TO_SOT_SMD:SOT-23-5, symbol Regulator_Linear:XC6210B332MR
- added U5: TC2185-1.8VxCTTR, Package_TO_SOT_SMD:SOT-23-5, symbol Regulator_Linear:TC2185-1.8VxCTTR
Connections:
- new net: C5.1, U5.1 (VIN), U5.3 (ON/~{OFF})
- new net: C6.1, U5.5 (VOUT)
- new net: C2.1, U3.5 (VOUT)
- new net: R1.1, U1.2 (PROG)
- new net: C3.1, U4.5 (VOUT)
- new net GND: C1.2, C2.2, C3.2, C4.2, C5.2, C6.2, J4.2, R1.2, U1.3 (GND), U1.9 (EPAD), U3.2 (GND), U4.2 (GND), U5.2 (GND)
- new net VCC: C1.1, U1.4 (V_{CC}), U3.1 (VIN), U3.3 (CE)
- new net V_BAT: C4.1, J4.1, U1.5 (BAT), U4.1 (VIN), U4.3 (CE)
- no-connect marks 0 -> 2
