File: Layout/Microcontroller.kicad_sch (KiCad schematic)
At the start: 0 parts

Commit message: First ICs Placed$
Parts:
- added J1: Conn_01x06_Pin(Stlink), Connector_PinHeader_2.54mm:PinHeader_1x01_P2.54mm_Vertical, symbol Connector:Conn_01x06_Pin
- added J2: Conn_01x07_Pin(Display), symbol Connector:Conn_01x07_Pin
- added U2: STM32L4Q5CGTx, Package_QFP:LQFP-48_7x7mm_P0.5mm, symbol MCU_ST_STM32L4:STM32L4Q5CGTx
Connections:
- new net: U2.23 (VSS), U2.35 (VSS), U2.47 (VSS)

Commit message: Routine Commit, small changes in schematic
Parts:
- removed J1: Conn_01x06_Pin(Stlink), Connector_PinHeader_2.54mm:PinHeader_1x01_P2.54mm_Vertical, symbol Connector:Conn_01x06_Pin
- added C7: C, symbol Device:C
- added IC1: OPT3101RHFR, ToF Driver:QFN50P400X500X100-29N-D, symbol OPT3101RHFR:OPT3101RHFR
- added J1: Conn_01x07_MountingPin, symbol Connector_Generic_MountingPin:Conn_01x07_MountingPin
- added J3: USB_B_Micro, symbol Connector:USB_B_Micro
- added R10, R11, R12, R13, R2, R3, R4, R5, R6, R7, R8, R9: R, symbol Device:R
- added SW1, SW2: SW_Omron_B3FS, symbol Switch:SW_Omron_B3FS
- added U6: USBLC6-2SC6, Package_TO_SOT_SMD:SOT-23-6, symbol Power_Protection:USBLC6-2SC6
Connections:
- net I2C2_SDA: now reaches J2.4 (Pin_4)
- net I2C2_SDA: now also U2.22 (PB11), R6.2
- net I2C2_SCL: now reaches J2.5 (Pin_5)
- net I2C2_SCL: now also U2.21 (PB10), R5.2
- net VCC: now reaches J2.6 (Pin_6)
- net VCC: now also J1.1 (Pin_1), J3.1 (VBUS), R12.1, R13.2, R7.1, R8.1, U6.5 (VBUS)
- net GND: now reaches J2.7 (Pin_7)
- net GND: now also U2.23 (VSS), U2.35 (VSS), U2.47 (VSS), U2.8 (VSSA), C7.2, J1.7 (Pin_7), J1.MP (MountPin), J3.5 (GND), J3.6 (Shield), R11.2, R2.1, R3.1, R4.1, SW1.1, U6.2 (GND)
- net 3V3: now reaches U2.24 (VDD)
- net 3V3: now also U2.36 (VDDUSB), U2.48 (VDD), U2.9 (VDDA), R10.2, R5.1, R6.1
- net at U2.30 (PA9): now also R13.1
- net at U2.32 (PA11): now also U6.1 (I/O1)
- net at U2.33 (PA12): now also U6.3 (I/O2)
- net JTMS: now reaches U2.34 (PA13)
- net JTMS: now also J1.2 (Pin_2)
- net JTCK: now reaches U2.37 (PA14)
- net JTCK: now also J1.3 (Pin_3)
- net JTDI: now reaches U2.38 (PA15)
- net JTDI: now also J1.5 (Pin_5)
- net JTDO: now reaches U2.39 (PB3)
- net JTDO: now also J1.4 (Pin_4)
- net nJRST: now reaches U2.40 (PB4)
- net nJRST: now also J1.6 (Pin_6)
- net I2C1_SCL: now reaches U2.42 (PB6)
- net I2C1_SCL: now also IC1.13 (SCL_S), R8.2
- net I2C1_SDA: now reaches U2.43 (PB7)
- net I2C1_SDA: now also IC1.14 (SDA_S), R7.2
- net at U2.7 (NRST): now also C7.1, R9.2
- new net: IC1.2 (A2), R4.2
- new net: J3.4 (ID), R11.1, R12.2
- new net: R10.1, R9.1, SW1.2
- new net: IC1.1 (A1), R3.2
- new net: IC1.28 (A0), R2.2
- new net: J3.2 (D-), U6.6 (I/O1)
- new net: J3.3 (D+), U6.4 (I/O2)
- new net REG_MODE: IC1.18 (REG_MODE)
- new net RST_MS: IC1.17 (~{RST_MS})
- new net SCL_M: IC1.15 (SCL_M)
- new net SDA_M: IC1.16 (SDA_M)
- no-connect marks 0 -> 3
Other:
- moved on the sheet: J2, U2

Commit message: Layout merged together
Parts:
- removed IC1: OPT3101RHFR, ToF Driver:QFN50P400X500X100-29N-D, symbol OPT3101RHFR:OPT3101RHFR
- removed R4, R5, R6, R7, R8: R, symbol Device:R
- removed SW2: SW_Omron_B3FS, symbol Switch:SW_Omron_B3FS
- added C8: C, symbol Device:C
- added SW3: SW_Omron_B3FS, symbol Switch:SW_Omron_B3FS
- added U7, U8, U9: VL53L0CXV0DH1, Sensor_Distance:ST_VL53L1x, symbol Sensor_Distance:VL53L0CXV0DH1
Connections:
- net 3V3: now also R2.2; no longer U2.24 (VDD), U2.36 (VDDUSB), U2.48 (VDD), U2.9 (VDDA)
- net GND: now also C8.2, SW3.1, U7.12 (GND), U7.2 (AVSSVCSEL), U7.3 (GND), U7.4 (GND), U7.6 (GND), U8.12 (GND), U8.2 (AVSSVCSEL), U8.3 (GND), U8.4 (GND), U8.6 (GND), U9.12 (GND), U9.2 (AVSSVCSEL), U9.3 (GND), U9.4 (GND), U9.6 (GND); no longer R2.1, R3.1
- net I2C1_SCL: now also J2.5 (Pin_5), U7.10 (SCL)
- net I2C1_SDA: now also J2.4 (Pin_4), U7.9 (SDA)
- net I2C2_SCL: now also U2.26 (PB13), U9.10 (SCL); no longer J2.5 (Pin_5), U2.21 (PB10)
- net I2C2_SDA: now also U2.27 (PB14), U9.9 (SDA); no longer J2.4 (Pin_4), U2.22 (PB11)
- net BTN: now reaches R3.2
- net BTN: now also U2.10 (PA0), C8.1
- net SHUT_TOF3: now reaches U2.20 (PB2)
- net SHUT_TOF3: now also U8.5 (XSHUT)
- net INT_TOF3: now reaches U2.25 (PB12)
- net INT_TOF3: now also U8.7 (GPIO1)
- net INT_TOF2: now reaches U2.28 (PB15)
- net INT_TOF2: now also U9.7 (GPIO1)
- net SHUT_TOF2: now reaches U2.41 (PB5)
- net SHUT_TOF2: now also U9.5 (XSHUT)
- net INT_TOF1: now reaches U2.45 (PB8)
- net INT_TOF1: now also U7.7 (GPIO1)
- net SHUT_TOF1: now reaches U2.46 (PB9)
- net SHUT_TOF1: now also U7.5 (XSHUT)
- net NRST: now reaches C7.1, R9.2, U2.7 (NRST)
- new net: R2.1, R3.1, SW3.2
- new net +3.3V: U2.24 (VDD), U2.36 (VDDUSB), U2.48 (VDD), U2.9 (VDDA), U7.1 (AVDDVCSEL), U7.11 (AVDD), U8.1 (AVDDVCSEL), U8.11 (AVDD), U9.1 (AVDDVCSEL), U9.11 (AVDD)
- new net I2C4_SCL: U2.21 (PB10), U8.10 (SCL)
- new net I2C4_SDA: U2.22 (PB11), U8.9 (SDA)
Other:
- note added: "-Buzzer -Debug Led -NOE -VOLTAGE -General -Gyroscope -Target laser"
- moved on the sheet: C7, J1, J2, J3, R10, R11, R12, R13, R9, SW1, U6
