File: Layout/Layout.kicad_pcb (KiCad board)
At the start: 2 copper layers, 50.5 x 26 mm, 1 part, among them IC1 OPT3101RHFR

Commit message: Started with Layout
Parts:
- added C1: 1uF, Capacitor_SMD:C_0603_1608Metric, F.Cu at (67.7, 35.7)
- added C10: 100nF, Capacitor_SMD:C_0603_1608Metric, F.Cu at (72.3, 40.1)
- added C12: 100nF, Capacitor_SMD:C_0603_1608Metric, F.Cu at (42.2, 45.9)
- added C13: 47nF, Capacitor_SMD:C_0603_1608Metric, F.Cu at (64.5, 68.0)
- added C14: 10uF, Capacitor_SMD:C_0603_1608Metric, F.Cu at (64.5, 64.5)
- added C15: 100nF, Capacitor_SMD:C_0603_1608Metric, F.Cu at (66.5, 64.5)
- added C16: 100nF, Capacitor_SMD:C_0603_1608Metric, F.Cu at (137.0, 43.2)
- added C17: 100nF, Capacitor_SMD:C_0603_1608Metric, F.Cu at (164.5, 96.5)
- added C18: n/a, Capacitor_SMD:C_0603_1608Metric, F.Cu at (137.0, 48.2)
- added C19: 100nF, Capacitor_SMD:C_0603_1608Metric, F.Cu at (44.7, 51.9)
- added C2: 1uF, Capacitor_SMD:C_0603_1608Metric, F.Cu at (67.7, 38.2)
- added C3: 100nF, Capacitor_SMD:C_0603_1608Metric, F.Cu at (178.5, 97.5)
- added C5: 100nF, Capacitor_SMD:C_0603_1608Metric, F.Cu at (202.0, 82.5)
- added C6: 100nF, Capacitor_SMD:C_0603_1608Metric, F.Cu at (206.0, 85.5)
- added C7: 100nF, Capacitor_SMD:C_0603_1608Metric, F.Cu at (191.0, 102.5)
- added C8: 100nF, Capacitor_SMD:C_0603_1608Metric, F.Cu at (202.0, 104.5)
- added C9: 100nF, Capacitor_SMD:C_0603_1608Metric, F.Cu at (212.0, 54.5)
- added D1: YELLOW LED, LED_SMD:LED_0603_1608Metric, F.Cu at (215.0, 95.8)
- added D2: BLUE LED, LED_SMD:LED_0603_1608Metric, F.Cu at (217.5, 96.0)
- added D3: RLD65NZN5-00A, Laser:RLD65NZN500A, F.Cu at (141.5, 31.0)
- added D4: BLUE LED, LED_SMD:LED_0603_1608Metric, F.Cu at (220.0, 96.0)
- added D5: BLUE LED, LED_SMD:LED_0603_1608Metric, F.Cu at (223.0, 96.0)
- added G1: Laser_Warnschild, Laser:Laser_Warnschild, F.Cu at (136.6, 56.9)
- added IC2: MAX4231AUT+T, Package_TO_SOT_SMD:SOT-23-6, F.Cu at (128.4, 31.8)
- added IC3: STM32F042G4U6, uC:uC_Footprint, F.Cu at (174.0, 97.0)
- added J1: Conn_01x07_Pin, Connector_PinHeader_2.54mm:PinHeader_1x07_P2.54mm_Vertical_SMD_Pin1Left, F.Cu at (198.9, 54.7)
- added J2: USB_B_Micro, Connector_USB:USB_Micro-B_Amphenol_10118193-0001LF_Horizontal, F.Cu at (37.3, 60.9)
- added J3: Conn_01x03_Pin, Connector_PinHeader_2.54mm:PinHeader_1x03_P2.54mm_Vertical_SMD_Pin1Left, F.Cu at (96.8, 59.0)
- added J4: Conn_01x04_Pin, Connector_PinHeader_2.54mm:PinHeader_1x04_P2.54mm_Vertical_SMD_Pin1Left, F.Cu at (89.6, 60.2)
- added R1: 330R, Resistor_SMD:R_0603_1608Metric, F.Cu at (215.0, 92.0)
- added R10: 10k, Resistor_SMD:R_0603_1608Metric, F.Cu at (191.0, 106.5)
- added R11: n/a, Resistor_SMD:R_0603_1608Metric, F.Cu at (50.2, 45.9)
- added R12: n/a, Resistor_SMD:R_0603_1608Metric, F.Cu at (50.2, 48.4)
- added R13: shunt, Resistor_SMD:R_2512_6332Metric, F.Cu at (46.0, 64.0)
- added R14: 0R, Resistor_SMD:R_0603_1608Metric, F.Cu at (145.1, 40.7)
- added R15: 0R, Resistor_SMD:R_0603_1608Metric, F.Cu at (62.0, 62.5)
- added R16: 4.7k, Resistor_SMD:R_0603_1608Metric, F.Cu at (145.1, 45.7)
- added R18: n/a, Resistor_SMD:R_0603_1608Metric, F.Cu at (199.5, 60.5)
- added R19: n/a, Resistor_SMD:R_0603_1608Metric, F.Cu at (203.0, 60.5)
- added R2: 10k, Resistor_SMD:R_0603_1608Metric, F.Cu at (202.0, 106.5)
- added R3: 10k, Resistor_SMD:R_0603_1608Metric, F.Cu at (202.0, 102.5)
- added R4: 0R, Resistor_SMD:R_0603_1608Metric, F.Cu at (72.0, 43.6)
- added R5: 390R, Resistor_SMD:R_0603_1608Metric, F.Cu at (217.5, 92.2)
- added R6: 390R, Resistor_SMD:R_0603_1608Metric, F.Cu at (220.0, 92.2)
- added R7: 390R, Resistor_SMD:R_0603_1608Metric, F.Cu at (223.0, 92.2)
- added R8: 0R, Resistor_SMD:R_0603_1608Metric, F.Cu at (64.9, 58.3)
- added R9: 10k, Resistor_SMD:R_0603_1608Metric, F.Cu at (191.0, 104.5)
- added RN1: 100R 4x0603, Resistor_SMD:R_Array_Concave_4x0603, F.Cu at (157.0, 46.0)
- added SW1: SW_Omron_B3FS, Button_Switch_SMD:SW_SPST_B3S-1000, F.Cu at (196.5, 104.5)
- added SW3: SW_Omron_B3FS, Button_Switch_SMD:SW_SPST_B3S-1000, F.Cu at (207.5, 104.5)
- added TR1: 2N7002AQ-7, Package_TO_SOT_SMD:SOT-23-3, F.Cu at (128.4, 36.4)
- added U2: AD8293G160ARJZ-R7, Package_TO_SOT_SMD:SOT-23-8, F.Cu at (59.5, 66.5)
- added U3: XC6210B332MR, Package_TO_SOT_SMD:SOT-23-5, F.Cu at (67.4, 43.5)
- added U4: ~, Package_TO_SOT_SMD:SOT-23-6, F.Cu at (128.4, 45.7)
- added U6: USBLC6-2SC6, Package_TO_SOT_SMD:SOT-23-6, F.Cu at (49.0, 59.5)
- added Y1: SG-210STF_48.0000ML5, Oszi:SG210STF480000ML5, F.Cu at (168.0, 96.5)
- IC1: value OPT3101RHFR -> VL53L4CDV0DH_1; footprint ToF Driver:QFN50P400X500X100-29N-D -> VL53L4CDV0DH/1:VL53L4CDV0DH1
- moved IC1 117.3 mm to (202.6, 87.1), turned to 90 degrees
Connections:
- IC1 pad 1: unconnected-(IC1-A1-Pad1) -> +3.3V
- IC1 pad 10: unconnected-(IC1-IOVDD_2-Pad10) -> /I2C1_SCL
- IC1 pad 11: unconnected-(IC1-GP1-Pad11) -> +3.3V
- IC1 pad 12: unconnected-(IC1-GP2-Pad12) -> GND
- IC1 pad 13: unconnected-(IC1-SCL_S-Pad13) -> +3.3V
- IC1 pad 2: unconnected-(IC1-A2-Pad2) -> GND
- IC1 pad 3: unconnected-(IC1-IOVSS_1-Pad3) -> GND
- IC1 pad 4: unconnected-(IC1-TX2-Pad4) -> GND
- IC1 pad 5: unconnected-(IC1-TX1-Pad5) -> /SHUT_TOF1
- IC1 pad 6: unconnected-(IC1-VSSL-Pad6) -> GND
- IC1 pad 7: unconnected-(IC1-TX0-Pad7) -> /INT_TOF1
- IC1 pad 9: unconnected-(IC1-IOVDD_1-Pad9) -> /I2C1_SDA
Other:
- board size 50.5 x 26 mm -> 75 x 50 mm

Commit message: Temporary commit before Atoplace usage
Parts:
- removed C13: 47nF, Capacitor_SMD:C_0603_1608Metric
- removed C15: 100nF, Capacitor_SMD:C_0603_1608Metric
- removed D3: RLD65NZN5-00A, Laser:RLD65NZN500A
- removed IC2: MAX4231AUT+T, Package_TO_SOT_SMD:SOT-23-6
- removed U2: AD8293G160ARJZ-R7, Package_TO_SOT_SMD:SOT-23-8
- added C11: 100nF, Capacitor_SMD:C_0402_1005Metric, F.Cu at (76.2, 84.3)
- added C4: 100nF, Capacitor_SMD:C_0402_1005Metric, F.Cu at (74.6, 93.0)
- added D7: RLD65NZN5-00A, Laser:RLD65NZN500A, F.Cu at (59.5, 90.8)
- added IC4: MAX4231AUT+T, Package_TO_SOT_SMD:SOT-23-6, F.Cu at (63.6, 98.5)
- added R21: 1k, Resistor_SMD:R_0402_1005Metric, F.Cu at (59.6, 100.0)
- added TP1: Testpoint, TestPoint:TestPoint_Pad_D1.0mm, F.Cu at (72.5, 97.2)
- added TP10: TestPoint, TestPoint:TestPoint_Pad_D1.0mm, F.Cu at (48.5, 77.5)
- added TP11: TestPoint, TestPoint:TestPoint_Pad_D1.0mm, F.Cu at (48.5, 75.2)
- added TP12: Testpoint, TestPoint:TestPoint_Pad_D1.0mm, F.Cu at (54.8, 98.8)
- added TP14: Testpoint, TestPoint:TestPoint_Pad_D1.0mm, F.Cu at (54.2, 80.8)
- added TP15: Testpoint, TestPoint:TestPoint_Pad_D1.0mm, F.Cu at (100.5, 73.0)
- added TP16: Testpoint, TestPoint:TestPoint_Pad_D1.0mm, F.Cu at (48.0, 102.5)
- added TP2: Testpoint, TestPoint:TestPoint_Pad_D1.0mm, F.Cu at (152.0, 79.4)
- added TP3: Testpoint, TestPoint:TestPoint_Pad_D1.0mm, F.Cu at (58.8, 85.8)
- added TP4: Testpoint, TestPoint:TestPoint_Pad_D1.0mm, F.Cu at (56.2, 85.8)
- added TP5: Testpoint, TestPoint:TestPoint_Pad_D1.0mm, F.Cu at (73.0, 89.2)
- added TP6: Testpoint, TestPoint:TestPoint_Pad_D1.0mm, F.Cu at (73.6, 79.6)
- added TP7: Testpoint, TestPoint:TestPoint_Pad_D1.0mm, F.Cu at (53.8, 85.8)
- added TP8: Testpoint, TestPoint:TestPoint_Pad_D1.0mm, F.Cu at (66.8, 102.0)
- added TP9: TestPoint, TestPoint:TestPoint_Pad_D1.0mm, F.Cu at (48.5, 80.0)
- added U1: INA197, Package_TO_SOT_SMD:SOT-23-5, F.Cu at (146.4, 85.2)
- C1, C10, C12, C14, C16, C17, C18, C19, C2, C3, C5, C6, C7, C8, C9: footprint Capacitor_SMD:C_0603_1608Metric -> Capacitor_SMD:C_0402_1005Metric
- J3: footprint Connector_PinHeader_2.54mm:PinHeader_1x03_P2.54mm_Vertical_SMD_Pin1Left -> Connector_PinHeader_2.54mm:PinHeader_1x03_P2.54mm_Vertical
- J4: footprint Connector_PinHeader_2.54mm:PinHeader_1x04_P2.54mm_Vertical_SMD_Pin1Left -> Connector_PinHeader_2.54mm:PinHeader_1x04_P2.54mm_Vertical
- R1, R10, R11, R12, R18, R19, R2, R3, R5, R6, R7, R9: footprint Resistor_SMD:R_0603_1608Metric -> Resistor_SMD:R_0402_1005Metric
- R14: value 0R -> 470R; footprint Resistor_SMD:R_0603_1608Metric -> Resistor_SMD:R_0402_1005Metric
- R15: value 0R -> 10R; footprint Resistor_SMD:R_0603_1608Metric -> Resistor_SMD:R_0402_1005Metric
- R16: value 4.7k -> 8.2k; footprint Resistor_SMD:R_0603_1608Metric -> Resistor_SMD:R_0402_1005Metric
- R8: value 0R -> 680R; footprint Resistor_SMD:R_0603_1608Metric -> Resistor_SMD:R_0402_1005Metric
- Y1: value SG-210STF_48.0000ML5 -> SG-210STF_8.0000ML5
- moved C6 156.7 mm to (49.5, 93.0), turned to 90 degrees
- moved IC1 150.4 mm to (52.2, 91.8), turned to -90 degrees
- moved C5 149.8 mm to (52.7, 95.5), turned to 180 degrees
- moved SW3 149.0 mm to (58.8, 113.0)
- moved C8 138.5 mm to (63.8, 113.2)
- moved R2 138.5 mm to (63.8, 115.2)
- moved R3 138.5 mm to (63.8, 111.2)
- moved J2 131.8 mm to (167.5, 81.5), turned to 90 degrees
- moved SW1 128.0 mm to (68.8, 113.0)
- moved R7 122.3 mm to (102.5, 113.5)
- moved D5 122.3 mm to (102.5, 117.0)
- moved R6 120.9 mm to (101.0, 113.5)
- moved D4 120.8 mm to (101.0, 117.0)
- moved R5 119.9 mm to (99.5, 113.5)
- moved D2 119.8 mm to (99.5, 117.0)
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Connections:
- IC3 pad 13: unconnected-(IC3-PA7-Pad13) -> Net-(IC3-PA7)
- IC3 pad 19: /USB_DM -> /USB_D-
- IC3 pad 20: /USB_DP -> /USB_D+
- IC3 pad 8: unconnected-(IC3-PA2-Pad8) -> Net-(IC3-PA2)
- IC3 pad 9: unconnected-(IC3-PA3-Pad9) -> Net-(IC3-PA3)
- J2 pad 1: +5V -> /IN+_SHUNT
- J2 pad 2: /USB_DM -> Net-(J2-D-)
- J2 pad 3: /USB_DP -> Net-(J2-D+)
- J2 pad 5: /IN+_SHUNT -> GND
- R13 pad 2: GND -> +5V
- R14 pad 1: +5V -> Net-(IC4-IN+)
- R14 pad 2: Net-(D3-K_LD) -> GND
- R15 pad 1: Net-(U2-IN+) -> GND
- R15 pad 2: /IN+_SHUNT -> Net-(R15-Pad2)
- R16 pad 2: /PD_LASER -> Net-(R16-Pad2)
- R8 pad 1: Net-(U2-IN-) -> Net-(R16-Pad2)
- R8 pad 2: GND -> /PD_LASER
- TR1 pad 3: GND -> Net-(TR1-D)
- U6 pad 1: /USB_DM -> /USB_D-
- U6 pad 3: /USB_DP -> /USB_D+
- U6 pad 4: /USB_DP -> Net-(J2-D+)
- U6 pad 6: /USB_DM -> Net-(J2-D-)
Routing:
- net Net-(TR1-G): track 0.00 -> 2.82 mm
Other:
- board size 75 x 50 mm -> 70 x 50 mm

Commit message: Compact version
Parts:
- moved J2 121.0 mm to (47.8, 99.0), turned to -90 degrees
- moved R12 110.7 mm to (53.3, 101.6), turned to 90 degrees
- moved R11 108.7 mm to (54.3, 101.6), turned to -90 degrees
- moved R13 103.5 mm to (55.8, 96.5), turned to 0 degrees
- moved C19 100.6 mm to (58.7, 104.3), turned to 180 degrees
- moved U6 99.2 mm to (58.7, 102.0), turned to 0 degrees
- moved C1 93.7 mm to (61.0, 96.0), turned to -90 degrees
- moved TP2 91.3 mm to (61.5, 91.5), turned to 180 degrees
- moved U1 90.8 mm to (55.9, 92.2), turned to 180 degrees
- moved C12 89.8 mm to (63.3, 99.0), turned to 0 degrees
- moved U3 87.9 mm to (64.0, 96.5), turned to 0 degrees
- moved C14 84.9 mm to (58.8, 91.7), turned to -90 degrees
- moved C2 81.8 mm to (67.2, 96.5), turned to 0 degrees
- moved C10 80.6 mm to (67.2, 95.4), turned to 0 degrees
- moved R4 77.7 mm to (67.2, 93.8), turned to 0 degrees
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Other:
- board size 70 x 50 mm -> 66.2 x 40 mm

Commit message: Commit of STM32 uC Conifg and Production data
Parts:
- removed C19: 100nF, Capacitor_SMD:C_0402_1005Metric
- added C13: 100nF, Capacitor_SMD:C_0402_1005Metric, F.Cu at (153.6, 95.5)
- J2: footprint Connector_USB:USB_Micro-B_Amphenol_10118193-0001LF_Horizontal -> Project_Lib:USB_Micro-B_Amphenol_10118193-0001LF_Horizontal
- TP10, TP11, TP9: footprint TestPoint:TestPoint_Pad_D1.0mm -> TestPoint:TestPoint_Pad_2.5x2.5mm
- moved G1 134.3 mm to (161.2, 84.5)
- moved TP11 98.5 mm to (150.0, 81.6)
- moved TP10 97.1 mm to (146.4, 81.6)
- moved TP9 96.0 mm to (142.8, 81.6)
- moved D1 92.2 mm to (138.5, 81.8), turned to -90 degrees
- moved J3 91.5 mm to (137.3, 114.4), turned to 0 degrees
- moved D2 90.8 mm to (137.0, 81.8), turned to -90 degrees
- moved D4 89.4 mm to (135.5, 81.8), turned to -90 degrees
- moved R1 88.6 mm to (138.5, 85.3), turned to 90 degrees
- moved D5 88.0 mm to (134.0, 81.8), turned to -90 degrees
- moved R5 87.1 mm to (137.0, 85.3), turned to 90 degrees
- moved R6 85.7 mm to (135.5, 85.3), turned to 90 degrees
- moved R7 84.2 mm to (134.0, 85.3), turned to 90 degrees
- moved J4 80.1 mm to (133.1, 122.0), turned to 180 degrees
- moved TP14 75.6 mm to (163.9, 111.6)
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Connections:
- IC3 pad 19: /USB_D- -> /USB1_2_D-
- IC3 pad 20: /USB_D+ -> /USB1_2_D+
- J2 pad 2: Net-(J2-D-) -> /USB1_1_D-
- J2 pad 3: Net-(J2-D+) -> /USB1_1_D+
- U6 pad 1: /USB_D- -> /USB1_1_D-
- U6 pad 3: /USB_D+ -> /USB1_1_D+
- U6 pad 4: Net-(J2-D+) -> /USB1_2_D+
- U6 pad 6: Net-(J2-D-) -> /USB1_2_D-
Routing:
- net +3.3V: track 0.00 -> 212.5 mm, vias 0 -> 8
- net GND: track 0.00 -> 66.9 mm, vias 0 -> 40
- net /I2C1_SDA: track 0.00 -> 64.3 mm, vias 0 -> 2
- net /I2C1_SCL: track 0.00 -> 63.1 mm, vias 0 -> 2
- net /SHUT_TOF1: track 0.00 -> 41.6 mm, vias 0 -> 4
- net /INT_TOF1: track 0.00 -> 41.4 mm
- net /PD_LASER: track 0.00 -> 38.6 mm, vias 0 -> 2
- net /U_SHUNT: track 0.00 -> 37.5 mm, vias 0 -> 2
- net +5V: track 0.00 -> 35.5 mm, vias 0 -> 2
- net Net-(IC3-PA2): track 0.00 -> 29.5 mm
- net Net-(IC3-PA7): track 0.00 -> 29.3 mm, vias 0 -> 2
- net /BTN: track 0.00 -> 28.4 mm, vias 0 -> 2
- net Net-(IC3-PA3): track 0.00 -> 28.1 mm
- net /DIM_LASER: track 0.00 -> 25.7 mm, vias 0 -> 2
- net /LED_USB: track 0.00 -> 23.6 mm, vias 0 -> 2
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- added copper zone on F.Cu, net +3.3V
- added copper zone on F.Cu, net +5V
- added copper zone on F.Cu, net /IN+_SHUNT
- added copper zone on B.Cu, net GND
- added copper zone on F.Cu, net GND
- added copper zone on F.Cu, net Net-(RN1-R1.2)
- added copper zone on F.Cu, net Net-(U3-VOUT)
Other:
- board size 66.2 x 40 mm -> 70 x 45.7 mm
- board text added: "3 2 1 USB"
- board text added: "NRST"
- board text added: "RA2"
- board text added: "RA3"
- board text added: "RA7"
