File: Layout/Layout.kicad_sch (KiCad schematic)
At the start: 57 parts, among them IC1 VL53L4CDV0DH_1, IC2 MAX4231AUT+T, IC3 STM32F042G4U6, J1 Conn_01x07_Pin, J2 USB_B_Micro, J3 Conn_01x03_Pin, J4 Conn_01x04_Pin, SW1 SW_Omron_B3FS, SW3 SW_Omron_B3FS, U2 AD8293G160ARJZ-R7, U3 XC6210B332MR, U6 USBLC6-2SC6, Y1 SG-210STF_48.0000ML5

Commit message: same
Parts:
- removed C13: 47nF, Capacitor_SMD:C_0603_1608Metric, symbol Device:C
- removed C15: 100nF, Capacitor_SMD:C_0603_1608Metric, symbol Device:C
- removed D3: RLD65NZN5-00A, Laser:RLD65NZN500A, symbol RLD65NZN5-00A:RLD65NZN5-00A
- removed IC2: MAX4231AUT+T, Package_TO_SOT_SMD:SOT-23-6, symbol MAX4231AUT+T:MAX4231AUT+T
- removed U2: AD8293G160ARJZ-R7, Package_TO_SOT_SMD:SOT-23-8, symbol 2026-10-10_13-37-23:AD8293G160ARJZ-R7
- added C11, C4: 100nF, Capacitor_SMD:C_0402_1005Metric, symbol Device:C
- added D7: RLD65NZN5-00A, Laser:RLD65NZN500A, symbol RLD65NZN5-00A:RLD65NZN5-00A
- added IC4: MAX4231AUT+T, Package_TO_SOT_SMD:SOT-23-6, symbol MAX4231AUT+T:MAX4231AUT+T
- added R21: 1k, Resistor_SMD:R_0402_1005Metric, symbol Device:R
- added TP1, TP12, TP14, TP15, TP16, TP2, TP3, TP4, TP5, TP6, TP7, TP8: Testpoint, TestPoint:TestPoint_Pad_D1.0mm, symbol Connector:TestPoint
- added TP10, TP11, TP9: TestPoint, TestPoint:TestPoint_Pad_D1.0mm, symbol Connector:TestPoint
- added U1: INA197, Package_TO_SOT_SMD:SOT-23-5, symbol Amplifier_Current:INA197
- C1, C10, C12, C14, C16, C17, C18, C19, C2, C3, C5, C6, C7, C8, C9: footprint Capacitor_SMD:C_0603_1608Metric -> Capacitor_SMD:C_0402_1005Metric
- J3: footprint Connector_PinHeader_2.54mm:PinHeader_1x03_P2.54mm_Vertical_SMD_Pin1Left -> Connector_PinHeader_2.54mm:PinHeader_1x03_P2.54mm_Vertical
- J4: footprint Connector_PinHeader_2.54mm:PinHeader_1x04_P2.54mm_Vertical_SMD_Pin1Left -> Connector_PinHeader_2.54mm:PinHeader_1x04_P2.54mm_Vertical
- R1, R10, R11, R12, R18, R19, R2, R3, R5, R6, R7, R9: footprint Resistor_SMD:R_0603_1608Metric -> Resistor_SMD:R_0402_1005Metric
- R14: value 0R -> 470R; footprint Resistor_SMD:R_0603_1608Metric -> Resistor_SMD:R_0402_1005Metric
- R15: value 0R -> 10R; footprint Resistor_SMD:R_0603_1608Metric -> Resistor_SMD:R_0402_1005Metric
- R16: value 4.7k -> 8.2k; footprint Resistor_SMD:R_0603_1608Metric -> Resistor_SMD:R_0402_1005Metric
- R8: value 0R -> 680R; footprint Resistor_SMD:R_0603_1608Metric -> Resistor_SMD:R_0402_1005Metric
- Y1: value SG-210STF_48.0000ML5 -> SG-210STF_8.0000ML5
Connections:
- net +3.3V: now also C11.1, C4.1, D7.3, IC4.6 (VDD), TP1.1, U1.3 (V+)
- net +5V: now also R13.2, U1.5 (-); no longer J2.1 (VBUS), R14.1
- net DIM_LASER: now also TP5.1
- net GND: now also J2.5 (GND), R14.2, R15.1, C11.2, C4.2, IC4.2 (VSS), TP14.1, TP15.1, TP16.1, U1.2 (GND); no longer R13.2, R8.2, TR1.3 (D)
- net I2C1_SCL: now also TP3.1
- net I2C1_SDA: now also TP4.1
- net IN+_SHUNT: now also J2.1 (VBUS), U1.4 (+); no longer J2.5 (GND), R15.2
- net INT_TOF1: now also TP7.1
- net PD_LASER: now also R8.2, IC4.4 (OUT), TP8.1; no longer R16.2
- net RCC_OSC_IN: now also TP6.1
- net USB_D+: no longer J2.3 (D+), U6.4 (I/O2)
- net USB_D-: no longer J2.2 (D-), U6.6 (I/O1)
- net U_SHUNT: now also TP2.1, U1.1
- net at R16.1: now also IC4.3 (IN-), R21.2
- net at IC3.13 (PA7): now also TP9.1
- net at IC3.8 (PA2): now also TP11.1
- net at IC3.9 (PA3): now also TP10.1
- net at R8.1: now also R16.2
- new net: D7.2, IC4.1 (IN+), R14.1, TP12.1
- new net: J2.2 (D-), U6.6 (I/O1)
- new net: J2.3 (D+), U6.4 (I/O2)
- new net: R15.2, R21.1
- new net: D7.1, TR1.3 (D)
- no-connect marks 9 -> 6
Other:
- note removed: "Display Connection"
- note removed: "Inst.Amp."
- note removed: "Microcontroller"
- note removed: "Oscillator"
- note removed: "PC-Connection"
- note removed: "Powersupply"
- note removed: "Targeting Laser + Photo Diode"
- note removed: "ToF Sensor"
- note removed: "f(U)=U/(160*R_SHUNT)= I_TOT"
- moved on the sheet: C1, C10, C12, C14, C16, C17, C18, C19, C2, C3, C5, C6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

Commit message: Commit of STM32 uC Conifg and Production data
Parts:
- removed C19: 100nF, Capacitor_SMD:C_0402_1005Metric, symbol Device:C
- removed J2: USB_B_Micro, Connector_USB:USB_Micro-B_Amphenol_10118193-0001LF_Horizontal, symbol Connector:USB_B_Micro
- added C13: 100nF, Capacitor_SMD:C_0402_1005Metric, symbol Device:C
- added J2: USB_B_Micro, Project_Lib:USB_Micro-B_Amphenol_10118193-0001LF_Horizontal, symbol Project_Lib:USB_B_Micro
- TP10, TP11, TP9: footprint TestPoint:TestPoint_Pad_D1.0mm -> TestPoint:TestPoint_Pad_2.5x2.5mm
Connections:
- net +3.3V: now also C13.1
- net GND: now also C13.2, J2.5 (GND)
- net IN+_SHUNT: now also J2.1 (VBUS)
- net USB1_2_D-: now reaches U6.6 (I/O1)
- net USB1_2_D-: now also IC3.19 (PA9/PA11)
- net USB1_2_D+: now reaches U6.4 (I/O2)
- net USB1_2_D+: now also IC3.20 (PA10/PA12)
- net at R11.1, R12.2: now also J2.4 (ID)
- net USB_D+ renamed USB1_1_D+
- net USB1_1_D+: now also J2.3 (D+); no longer IC3.20 (PA10/PA12)
- net USB_D- renamed USB1_1_D-
- net USB1_1_D-: now also J2.2 (D-); no longer IC3.19 (PA9/PA11)
Other:
- moved on the sheet: C12, R11
